Commit message: empty urdf

File: diffbot_navigation/urdf/diffbot.urdf.xacro (robot description, xacro)
@@ -2,298 +2,3 @@
 <robot xmlns:xacro="http://www.ros.org/wiki/xacro" name="diffbot">
     <xacro:include filename="materials.xacro" />
-    <!-- Constants -->
-    <xacro:property name="PI" value="3.14159265359" />
-    <xacro:property name="BASE_X" value="0.2" />
-    <xacro:property name="BASE_Y" value="0.2" />
-    <xacro:property name="BASE_Z" value="0.005" />
-    <xacro:property name="BASE_M" value="0.2" />
-    <xacro:property name="CASTER_OFF_X" value="-0.09" />
-    <xacro:property name="CASTER_OFF_Z" value="-0.03" />
-    <xacro:property name="CASTER_R" value="0.01" />
-    <xacro:property name="CASTER_M" value="0.1" />
-    <xacro:property name="WHEEL_OFF_X" value="0.075" />
-    <xacro:property name="WHEEL_OFF_Y" value="0.115" />
-    <xacro:property name="WHEEL_OFF_Z" value="-0.01" />
-    <xacro:property name="WHEEL_L" value="0.025" />
-    <xacro:property name="WHEEL_R" value="0.03" />
-    <xacro:property name="WHEEL_M" value="0.05" />
-    <xacro:property name="LIDAR_OFF_Z" value="0.05" />
-    <xacro:property name="LIDAR_R" value="0.035" />
-    <xacro:property name="LIDAR_L" value="0.02" />
-    <xacro:property name="LIDAR_M" value="0.17" />
-    <xacro:property name="CAM_OFF_X" value="0.1" />
-    <xacro:property name="CAM_OFF_Z" value="0.05" />
-    <xacro:property name="CAM_R" value="0.00425" />
-    <xacro:property name="CAM_L" value="0.001" />
-    <xacro:property name="CAM_M" value="0.005" />
-    <xacro:property name="IMU_OFF_X" value="0.075" />
-    <xacro:property name="IMU_X" value="0.03" />
-    <xacro:property name="IMU_Y" value="0.02" />
-    <xacro:property name="IMU_Z" value="0.02" />
-    <xacro:property name="IMU_M" value="0.005" />
-    <!-- Macros -->
-    <xacro:macro name="Wheel" params="prefix y_reflect">
-        <joint name="${prefix}_wheel_joint" type="continuous">
-            <parent link="base_link" />
-            <child link="${prefix}_wheel_link" />
-            <origin xyz="${WHEEL_OFF_X} ${y_reflect*WHEEL_OFF_Y} ${WHEEL_OFF_Z}" rpy="${-PI/2} 0 0" />
-            <axis xyz="0 0 1" />
-        </joint>
-        <link name="${prefix}_wheel_link">
-            <visual>
-                <geometry>
-                    <cylinder radius="${WHEEL_R}" length="${WHEEL_L}" />
-                </geometry>
-                <material name="black" />
-            </visual>
-            <collision>
-                <geometry>
-                    <cylinder radius="${WHEEL_R}" length="${WHEEL_L}" />
-                </geometry>
-            </collision>
-            <xacro:CylinderInertial m="${WHEEL_M}" r="${WHEEL_R}" l="${WHEEL_L}" />
-        </link>
-        <gazebo reference="${prefix}_wheel_link">
-            <material>Gazebo/Black</material>
-        </gazebo>
-    </xacro:macro>
-    <xacro:macro name="BoxInertial" params="m x y z">
-        <inertial>
-            <mass value="${m}" />
-            <inertia ixx="${(m/12) * (z*z + y*y)}" ixy="0.0" ixz="0.0" iyy="${(m/12) * (x*x + z*z)}" iyz="0.0" izz="${(m/12) * (y*y + x*x)}" />
-        </inertial>
-    </xacro:macro>
-    <xacro:macro name="CylinderInertial" params="m r l">
-        <inertial>
-            <mass value="${m}" />
-            <inertia ixx="${(m/12) * (3*r*r + l*l)}" ixy="0" ixz="0" iyy="${(m/12) * (3*r*r + l*l)}" iyz="0" izz="${(m/2) * (r*r)}" />
-        </inertial>
-    </xacro:macro>
-    <xacro:macro name="SphereInertial" params="m r">
-        <inertial>
-            <mass value="${m}" />
-            <inertia ixx="${(2/5) * m * (r*r)}" ixy="0.0" ixz="0.0" iyy="${(2/5) * m * (r*r)}" iyz="0.0" izz="${(2/5) * m * (r*r)}" />
-        </inertial>
-    </xacro:macro>
-    <!-- Start Modelling -->
-    <link name="base_link">
-        <visual>
-            <geometry>
-                <box size="${BASE_X} ${BASE_Y} ${BASE_Z}"/>
-            </geometry>
-            <material name="purple"/>
-        </visual>
-        <collision>
-            <geometry>
-                <box size="${BASE_X} ${BASE_Y} ${BASE_Z}"/>
-            </geometry>
-        </collision>
-        <xacro:BoxInertial m="${BASE_M}" x="${BASE_X}" y="${BASE_Y}" z="${BASE_Z}" />
-    </link>
-    <gazebo reference="base_link">
-        <material>Gazebo/Purple</material>
-    </gazebo>
-    <joint name="footprint_joint" type="fixed">
-        <parent link="base_link"/>
-        <child link="base_footprint"/>
-        <origin xyz="0 0 ${CASTER_OFF_Z - CASTER_R}"/>
-    </joint>
-    <link name="base_footprint">
-    </link>
-    <joint name="caster joint" type="fixed">
-        <parent link="base_link"/>
-        <child link="caster"/>
-        <origin xyz="${CASTER_OFF_X} 0 ${CASTER_OFF_Z}"/>
-    </joint>
-    <link name="caster">
-        <visual>
-            <geometry>
-                <sphere radius="${CASTER_R}"/>
-            </geometry>
-            <material name="gray"/>
-        </visual>
-        <collision>
-            <geometry>
-                <sphere radius="${CASTER_R}"/>
-            </geometry>
-        </collision>
-        <xacro:SphereInertial m="${CASTER_M}" r="${CASTER_R}" />
-    </link>
-    <gazebo reference="caster">
-        <mu1>0.0001</mu1>
-        <mu2>0.0001</mu2>
-        <material>Gazebo/Gray</material>
-    </gazebo>
-    <xacro:Wheel prefix="left" y_reflect="1" />
-    <xacro:Wheel prefix="right" y_reflect="-1" />
-    <gazebo>
-        <plugin name="differential_drive_controller" filename="libgazebo_ros_diff_drive.so">
-            <!-- wheels -->
-            <left_joint>left_wheel_joint</left_joint>
-            <right_joint>right_wheel_joint</right_joint>
-            <!-- kinematics -->
-            <wheel_separation>0.23</wheel_separation>
-            <wheel_diameter>0.06</wheel_diameter>
-            <!-- tfs -->
-            <publish_odom>true</publish_odom>
-            <publish_odom_tf>true</publish_odom_tf>
-            <publish_wheel_tf>true</publish_wheel_tf>
-            <odometry_frame>odom</odometry_frame>
-            <!-- limits -->
-            <max_wheel_torque>20</max_wheel_torque>
-            <max_acceleration>1.0</max_acceleration>
-            <!-- miscs -->
-            <robot_base_frame>base_link</robot_base_frame>
-            <update_rate>100</update_rate>
-        </plugin>
-    </gazebo>
-    <joint name="lidar_joint" type="fixed">
-        <parent link="base_link"/>
-        <child link="lidar"/>
-        <origin xyz="0 0 ${LIDAR_OFF_Z}"/>
-    </joint>
-    <link name="lidar">
-        <visual>
-            <geometry>
-                <cylinder radius="${LIDAR_R}" length="${LIDAR_L}" />
-            </geometry>
-            <material name="black" />
-        </visual>
-        <collision>
-            <geometry>
-                <cylinder radius="${LIDAR_R}" length="${LIDAR_L}" />
-            </geometry>
-        </collision>
-        <xacro:CylinderInertial m="${LIDAR_M}" r="${LIDAR_R}" l="${LIDAR_L}" />
-        <!-- <inertial>
-            <mass value="${LIDAR_M}" />
-            <inertia ixx="${(LIDAR_M/12) * (3*LIDAR_R*LIDAR_R + LIDAR_L*LIDAR_L)}" ixy="0" ixz="0" iyy="${(m/12) * (3*r*r + l*l)}" iyz="0" izz="${(LIDAR_M/2) * (LIDAR_R*LIDAR_R)}" />
-        </inertial> -->
-    </link>
-    <gazebo reference="lidar">
-        <material>Gazebo/Blue</material>
-        <sensor name="lidar" type="ray">
-            <always_on>true</always_on>
-            <visualize>true</visualize>
-            <update_rate>5</update_rate>
-            <ray>
-                <scan>
-                    <horizontal>
-                        <samples>360</samples>
-                        <resolution>1.000000</resolution>
-                        <min_angle>0.000000</min_angle>
-                        <max_angle>6.280000</max_angle>
-                    </horizontal>
-                </scan>
-                <range>
-                    <min>0.120000</min>
-                    <max>6</max>
-                    <resolution>0.015000</resolution>
-                </range>
-                <noise>
-                    <type>gaussian</type>
-                    <mean>0.0</mean>
-                    <stddev>0.01</stddev>
-                </noise>
-            </ray>
-            <plugin name="scan" filename="libgazebo_ros_ray_sensor.so">
-                <ros>
-                    <remapping>~/out:=scan</remapping>
-                </ros>
-                <output_type>sensor_msgs/LaserScan</output_type>
-                <frame_name>lidar</frame_name>
-            </plugin>
-        </sensor>
-    </gazebo>
-    <joint name="imu_joint" type="fixed">
-        <parent link="base_link"/>
-        <child link="imu"/>
-        <origin xyz="${IMU_OFF_X} 0 0"/>
-    </joint>
-    <link name="imu">
-        <visual>
-            <geometry>
-                <box size="${IMU_X} ${IMU_Y} ${IMU_Z}" />
-            </geometry>
-            <material name="green" />
-        </visual>
-        <collision>
-            <geometry>
-                <box size="${IMU_X} ${IMU_Y} ${IMU_Z}" />
-            </geometry>
-        </collision>
-        <xacro:BoxInertial m="${IMU_M}" x="${IMU_X}" y="${IMU_Y}" z="${IMU_Z}" />
-        <!-- <inertial>
-            <mass value="${LIDAR_M}" />
-            <inertia ixx="${(LIDAR_M/12) * (3*LIDAR_R*LIDAR_R + LIDAR_L*LIDAR_L)}" ixy="0" ixz="0" iyy="${(m/12) * (3*r*r + l*l)}" iyz="0" izz="${(LIDAR_M/2) * (LIDAR_R*LIDAR_R)}" />
-        </inertial> -->
-    </link>
-    <gazebo reference="imu">
-        <sensor name="imu_sensor" type="imu">
-         <plugin filename="libgazebo_ros_imu_sensor.so" name="imu_plugin">
-            <ros>
-              <remapping>~/out:=imu</remapping>
-            </ros>
-            <initial_orientation_as_reference>false</initial_orientation_as_reference>
-          </plugin>
-          <always_on>true</always_on>
-          <update_rate>100</update_rate>
-          <visualize>true</visualize>
-          <imu>
-            <angular_velocity>
-              <x>
-                <noise type="gaussian">
-                  <mean>0.0</mean>
-                  <stddev>2e-4</stddev>
-                  <bias_mean>0.0000075</bias_mean>
-                  <bias_stddev>0.0000008</bias_stddev>
-                </noise>
-              </x>
-              <y>
-                <noise type="gaussian">
-                  <mean>0.0</mean>
-                  <stddev>2e-4</stddev>
-                  <bias_mean>0.0000075</bias_mean>
-                  <bias_stddev>0.0000008</bias_stddev>
-                </noise>
-              </y>
-              <z>
-                <noise type="gaussian">
-                  <mean>0.0</mean>
-                  <stddev>2e-4</stddev>
-                  <bias_mean>0.0000075</bias_mean>
-                  <bias_stddev>0.0000008</bias_stddev>
-                </noise>
-              </z>
-            </angular_velocity>
-            <linear_acceleration>
-              <x>
-                <noise type="gaussian">
-                  <mean>0.0</mean>
-                  <stddev>1.7e-2</stddev>
-                  <bias_mean>0.1</bias_mean>
-                  <bias_stddev>0.001</bias_stddev>
-                </noise>
-              </x>
-              <y>
-                <noise type="gaussian">
-                  <mean>0.0</mean>
-                  <stddev>1.7e-2</stddev>
-                  <bias_mean>0.1</bias_mean>
-                  <bias_stddev>0.001</bias_stddev>
-                </noise>
-              </y>
-              <z>
-                <noise type="gaussian">
-                  <mean>0.0</mean>
-                  <stddev>1.7e-2</stddev>
-                  <bias_mean>0.1</bias_mean>
-                  <bias_stddev>0.001</bias_stddev>
-                </noise>
-              </z>
-            </linear_acceleration>
-          </imu>
-        </sensor>
-        <material>Gazebo/Green</material>
-      </gazebo>
 </robot>
